Commit message: rpy="0 0 180"

File: beerbot/beerbot_description/urdf/base.urdf.xacro (robot description, xacro)
@@ -28,5 +28,5 @@
     <link name="${parent}_${suffix}_wheel_link">
       <visual>
-        <origin xyz="0 0 0" rpy="0 0 0" />
+        <origin xyz="0 0 0" rpy="0 0 180" />
         <geometry>
           <cylinder radius="${wheel_radius}" length="${wheel_length}"/>
@@ -35,5 +35,5 @@
       </visual>
       <collision>
-        <origin xyz="0 0 0" rpy="0 0 0" />
+        <origin xyz="0 0 0" rpy="0 0 180" />
         <geometry>
           <cylinder radius="${wheel_radius}" length="${wheel_length}"/>
@@ -41,5 +41,5 @@
       </collision>
       <inertial>
-        <origin xyz="0 0 ${wheel_radius}" rpy="0 0 0"/>
+        <origin xyz="0 0 ${wheel_radius}" rpy="0 0 180"/>
         <mass value="0.2"/>
         <inertia
@@ -71,5 +71,5 @@
     <link name="${name}_link">
       <visual>
-        <origin xyz="0 0 ${ground_clearance}" rpy="0 0 0" />
+        <origin xyz="0 0 ${ground_clearance}" rpy="0 0 180" />
         <geometry>
           <!-- <mesh filename="package://beerbot_description/meshes/base.stl"  /> -->
@@ -79,5 +79,5 @@
       </visual>
       <visual>
-        <origin xyz="0 0 ${level1_clearance}" rpy="0 0 0" />
+        <origin xyz="0 0 ${level1_clearance}" rpy="0 0 180" />
         <geometry>
 	  <cylinder radius="${base_radius}" length="${base_length}"/>
@@ -86,5 +86,5 @@
       </visual>
       <visual>
-        <origin xyz="0 0 ${level2_clearance}" rpy="0 0 0" />
+        <origin xyz="0 0 ${level2_clearance}" rpy="0 0 180" />
         <geometry>
 	  <cylinder radius="${base_radius}" length="${base_length}"/>
@@ -93,5 +93,5 @@
       </visual>
       <visual>
-        <origin xyz="0 0 ${level3_clearance}" rpy="0 0 0" />
+        <origin xyz="0 0 ${level3_clearance}" rpy="0 0 180" />
         <geometry>
 	  <cylinder radius="${base_radius}" length="${base_length}"/>
@@ -117,5 +117,5 @@
       to keep lidar free for object detection (otherwise it would be blocked by collision object) -->
       <collision>
-      <origin xyz="0 0 ${level2_clearance/2}" rpy="0 0 0" />
+      <origin xyz="0 0 ${level2_clearance/2}" rpy="0 0 180" />
         <geometry>
           <cylinder radius="${base_collision_radius}" length="${level2_clearance}"/>
@@ -123,5 +123,5 @@
       </collision>
       <collision>
-        <origin xyz="0 0 ${level3_clearance+base_collision_top_clearance/2}" rpy="0 0 0" />
+        <origin xyz="0 0 ${level3_clearance+base_collision_top_clearance/2}" rpy="0 0 180" />
         <geometry>
           <cylinder radius="${base_collision_radius}" length="${base_collision_top_clearance}"/>
@@ -129,5 +129,5 @@
       </collision>
       <inertial>
-        <origin xyz="0 0 ${base_radius}" rpy="0 0 0"/>
+        <origin xyz="0 0 ${base_radius}" rpy="0 0 180"/>
         <mass value="5"/>
         <inertia

File: beerbot/beerbot_description/urdf/beerbot.urdf.xacro (robot description, xacro)
@@ -12,5 +12,5 @@
   <!-- Camera -->
   <kinect_camera name="head_camera" parent="base_link">
-    <origin xyz="0 0 0.35" rpy="0 0 0"/>
+    <origin xyz="0 0 0.35" rpy="0 0 180"/>
   </kinect_camera>
   <!-- extensions -->

File: beerbot/beerbot_description/urdf/kinect_camera.urdf.xacro (robot description, xacro)
@@ -11,5 +11,5 @@
         <inertial_sphere mass="0.01" diameter="0.07" />
         <visual>
-          <origin xyz="0 0 0" rpy="0 0 0" />
+          <origin xyz="0 0 0" rpy="0 0 180" />
           <geometry>
             <mesh filename="package://beerbot_description/meshes/kinect_camera_simple.dae"/>
@@ -17,5 +17,5 @@
         </visual>
         <collision>
-          <origin xyz="0 0 0" rpy="0 0 0" />
+          <origin xyz="0 0 0" rpy="0 0 180" />
           <geometry>
             <mesh filename="package://beerbot_description/meshes/kinect_camera_simple.stl"/>
@@ -24,5 +24,5 @@
       </link>
       <joint name="${name}_depth_joint" type="fixed">
-        <origin xyz="0.0 -0.02 0.0" rpy="0 0 0" />
+        <origin xyz="0.0 -0.02 0.0" rpy="0 0 180" />
         <parent link="${name}_link" />
         <child link="${name}_depth_frame"/>
@@ -36,5 +36,5 @@
       <link name="${name}_depth_optical_frame"/>
       <joint name="${name}_rgb_joint" type="fixed">
-        <origin xyz="0.0 -0.0125 0.0" rpy="0 0 0" />
+        <origin xyz="0.0 -0.0125 0.0" rpy="0 0 180" />
         <parent link="${name}_link" />
         <child link="${name}_rgb_frame"/>

File: beerbot/beerbot_description/urdf/lidar.urdf.xacro (robot description, xacro)
@@ -10,5 +10,5 @@
     <link name="${name}_link">
       <visual>
-        <origin xyz="0 0 -0.01718" rpy="0 0 0" />
+        <origin xyz="0 0 -0.01718" rpy="0 0 180" />
         <geometry>
 	  <!-- <mesh filename="package://frobo_description/meshes/lidar.stl" /> -->

Commit message: rpy="0 0 0"

File: beerbot/beerbot_description/urdf/base.urdf.xacro (robot description, xacro)
@@ -28,5 +28,5 @@
     <link name="${parent}_${suffix}_wheel_link">
       <visual>
-        <origin xyz="0 0 0" rpy="0 0 180" />
+        <origin xyz="0 0 0" rpy="0 0 0" />
         <geometry>
           <cylinder radius="${wheel_radius}" length="${wheel_length}"/>
@@ -35,5 +35,5 @@
       </visual>
       <collision>
-        <origin xyz="0 0 0" rpy="0 0 180" />
+        <origin xyz="0 0 0" rpy="0 0 0" />
         <geometry>
           <cylinder radius="${wheel_radius}" length="${wheel_length}"/>
@@ -41,5 +41,5 @@
       </collision>
       <inertial>
-        <origin xyz="0 0 ${wheel_radius}" rpy="0 0 180"/>
+        <origin xyz="0 0 ${wheel_radius}" rpy="0 0 0"/>
         <mass value="0.2"/>
         <inertia
@@ -71,5 +71,5 @@
     <link name="${name}_link">
       <visual>
-        <origin xyz="0 0 ${ground_clearance}" rpy="0 0 180" />
+        <origin xyz="0 0 ${ground_clearance}" rpy="0 0 0" />
         <geometry>
           <!-- <mesh filename="package://beerbot_description/meshes/base.stl"  /> -->
@@ -79,5 +79,5 @@
       </visual>
       <visual>
-        <origin xyz="0 0 ${level1_clearance}" rpy="0 0 180" />
+        <origin xyz="0 0 ${level1_clearance}" rpy="0 0 0" />
         <geometry>
 	  <cylinder radius="${base_radius}" length="${base_length}"/>
@@ -86,5 +86,5 @@
       </visual>
       <visual>
-        <origin xyz="0 0 ${level2_clearance}" rpy="0 0 180" />
+        <origin xyz="0 0 ${level2_clearance}" rpy="0 0 0" />
         <geometry>
 	  <cylinder radius="${base_radius}" length="${base_length}"/>
@@ -93,5 +93,5 @@
       </visual>
       <visual>
-        <origin xyz="0 0 ${level3_clearance}" rpy="0 0 180" />
+        <origin xyz="0 0 ${level3_clearance}" rpy="0 0 0" />
         <geometry>
 	  <cylinder radius="${base_radius}" length="${base_length}"/>
@@ -117,5 +117,5 @@
       to keep lidar free for object detection (otherwise it would be blocked by collision object) -->
       <collision>
-      <origin xyz="0 0 ${level2_clearance/2}" rpy="0 0 180" />
+      <origin xyz="0 0 ${level2_clearance/2}" rpy="0 0 0" />
         <geometry>
           <cylinder radius="${base_collision_radius}" length="${level2_clearance}"/>
@@ -123,5 +123,5 @@
       </collision>
       <collision>
-        <origin xyz="0 0 ${level3_clearance+base_collision_top_clearance/2}" rpy="0 0 180" />
+        <origin xyz="0 0 ${level3_clearance+base_collision_top_clearance/2}" rpy="0 0 0" />
         <geometry>
           <cylinder radius="${base_collision_radius}" length="${base_collision_top_clearance}"/>
@@ -129,5 +129,5 @@
       </collision>
       <inertial>
-        <origin xyz="0 0 ${base_radius}" rpy="0 0 180"/>
+        <origin xyz="0 0 ${base_radius}" rpy="0 0 0"/>
         <mass value="5"/>
         <inertia

File: beerbot/beerbot_description/urdf/beerbot.urdf.xacro (robot description, xacro)
@@ -12,5 +12,5 @@
   <!-- Camera -->
   <kinect_camera name="head_camera" parent="base_link">
-    <origin xyz="0 0 0.35" rpy="0 0 180"/>
+    <origin xyz="0 0 0.35" rpy="0 0 0"/>
   </kinect_camera>
   <!-- extensions -->

File: beerbot/beerbot_description/urdf/kinect_camera.urdf.xacro (robot description, xacro)
@@ -11,5 +11,5 @@
         <inertial_sphere mass="0.01" diameter="0.07" />
         <visual>
-          <origin xyz="0 0 0" rpy="0 0 180" />
+          <origin xyz="0 0 0" rpy="0 0 1.57" />
           <geometry>
             <mesh filename="package://beerbot_description/meshes/kinect_camera_simple.dae"/>
@@ -17,5 +17,5 @@
         </visual>
         <collision>
-          <origin xyz="0 0 0" rpy="0 0 180" />
+          <origin xyz="0 0 0" rpy="0 0 1.57" />
           <geometry>
             <mesh filename="package://beerbot_description/meshes/kinect_camera_simple.stl"/>
@@ -24,5 +24,5 @@
       </link>
       <joint name="${name}_depth_joint" type="fixed">
-        <origin xyz="0.0 -0.02 0.0" rpy="0 0 180" />
+        <origin xyz="0.0 -0.02 0.0" rpy="0 0 1.57" />
         <parent link="${name}_link" />
         <child link="${name}_depth_frame"/>
@@ -36,5 +36,5 @@
       <link name="${name}_depth_optical_frame"/>
       <joint name="${name}_rgb_joint" type="fixed">
-        <origin xyz="0.0 -0.0125 0.0" rpy="0 0 180" />
+        <origin xyz="0.0 -0.0125 0.0" rpy="0 0 1.57" />
         <parent link="${name}_link" />
         <child link="${name}_rgb_frame"/>

File: beerbot/beerbot_description/urdf/lidar.urdf.xacro (robot description, xacro)
@@ -10,5 +10,5 @@
     <link name="${name}_link">
       <visual>
-        <origin xyz="0 0 -0.01718" rpy="0 0 180" />
+        <origin xyz="0 0 -0.01718" rpy="0 0 0" />
         <geometry>
 	  <!-- <mesh filename="package://frobo_description/meshes/lidar.stl" /> -->
